Commit message: Add parametrized .xacro files for every sensor and white QR calibration target, with spawnable versions from .launch files.

File: gazebo_models/blackflys/monocular_sensor.urdf.xacro (robot description, xacro)
@@ -1,7 +1,8 @@
 <?xml version="1.0"?>
 <robot xmlns:xacro="http://www.ros.org/wiki/xacro" name="monocular_sensor">
-<xacro:macro name="monocular_sensor" params="name hfov hz **resolution">
+<xacro:macro name="monocular_sensor" params="name hfov hz noise **resolution">
   <gazebo reference="${name}_link">
-    <turnGravityOff>true</turnGravityOff>
+    <static>true</static>
+    <turnGravityOff>false</turnGravityOff>
     <sensor name="zoe_narrow_link_camera" type="camera">
       <camera>
@@ -18,5 +19,5 @@
           <type>gaussian</type>
           <mean>0.0</mean>
-          <stddev>0.007</stddev>
+          <stddev>${noise}</stddev>
         </noise>
       </camera>

File: gazebo_models/calibration_whiteqr_pattern/calibration_whiteqr.urdf.xacro (robot description, xacro)
@@ -1,6 +1,5 @@
 <?xml version="1.0"?>
-<robot xmlns:xacro="http://www.ros.org/wiki/xacro" name="monocular_cam">
-  <xacro:include filename="$(find velo2cam_gazebo)/../gazebo_models//blackflys/monocular_sensor.urdf.xacro"/>
-  <xacro:macro name="blackflys" params="parent name hfov hz noise *origin *resolution">
+<robot xmlns:xacro="http://www.ros.org/wiki/xacro" name="calibration_whiteqr">
+<xacro:macro name="calibration_whiteqr" params="parent name *origin">
    <!-- Base Link -->
     <joint name="${name}_base_mount_joint" type="fixed">
@@ -17,20 +16,17 @@
       <collision name="collision">
         <geometry>
-          <mesh filename="model://blackflys/meshes/blackflys.stl" />
+          <mesh filename="model://calibration_whiteqr_pattern/meshes/whitebig.stl" />
         </geometry>
       </collision>
       <visual name="visual">
         <geometry>
-          <mesh filename="model://blackflys/meshes/blackflys.dae" />
+          <mesh filename="model://calibration_whiteqr_pattern/meshes/whitebig.dae" />
         </geometry>
       </visual>
     </link>
-    <monocular_sensor name="${name}" hfov="${hfov}" hz="${hz}" noise="${noise}">
-      <xacro:insert_block name="resolution" />
-    </monocular_sensor>
     <gazebo reference="${name}_link">
       <static>true</static>
       <turnGravityOff>false</turnGravityOff>
     </gazebo>
-  </xacro:macro>
+</xacro:macro>
 </robot>

File: gazebo_models/velodyne_HDL32/hdl32.urdf.xacro (robot description, xacro)
@@ -1,5 +1,5 @@
 <?xml version="1.0"?>
 <robot xmlns:xacro="http://www.ros.org/wiki/xacro" name="hdl32">
-	<xacro:macro name="hdl32" params="parent name hz *origin">
+	<xacro:macro name="hdl32" params="parent name hz *origin noise:=0.008">
 	    <joint name="${name}_base_mount_joint" type="fixed">
 	      <xacro:insert_block name="origin" />
@@ -29,4 +29,5 @@
     	</link>
 	    <gazebo reference="${name}_link">
+      		<static>true</static>
 	      <turnGravityOff>false</turnGravityOff>
 	      <sensor name='velodyne-HDL32' type='ray'>
@@ -60,9 +61,9 @@
 	          </ray>
 	          <plugin name='gazebo_ros_laser_controller' filename='libgazebo_ros_velodyne_laser.so'>
-	            <topicName>/velodyne_points</topicName>
+	            <topicName>/${name}_points</topicName>
 	            <frameName>${name}</frameName>
 	            <min_range>0.9</min_range>
 	            <max_range>70.0</max_range>
-	            <gaussianNoise>0.008</gaussianNoise>
+	            <gaussianNoise>${noise}</gaussianNoise>
 	            <robotNamespace>/</robotNamespace>
 	          </plugin>

File: gazebo_models/velodyne_HDL64/hdl64.urdf.xacro (robot description, xacro)
@@ -1,5 +1,5 @@
 <?xml version="1.0"?>
 <robot xmlns:xacro="http://www.ros.org/wiki/xacro" name="hdl64">
-	<xacro:macro name="hdl64" params="parent name hz *origin">
+	<xacro:macro name="hdl64" params="parent name hz *origin noise:=0.008">
 	    <joint name="${name}_base_mount_joint" type="fixed">
 	      <xacro:insert_block name="origin" />
@@ -23,4 +23,5 @@
     	</link>
 	    <gazebo reference="${name}_link">
+      		<static>true</static>
 	      <turnGravityOff>false</turnGravityOff>
 	      <sensor name='velodyne-HDL64' type='ray'>
@@ -54,9 +55,9 @@
 	          </ray>
 	          <plugin name='gazebo_ros_laser_controller' filename='libgazebo_ros_velodyne_laser.so'>
-	            <topicName>/velodyne_points</topicName>
+	            <topicName>/${name}_points</topicName>
 	            <frameName>${name}</frameName>
 	            <min_range>0.9</min_range>
 	            <max_range>70.0</max_range>
-	            <gaussianNoise>0.008</gaussianNoise>
+	            <gaussianNoise>${noise}</gaussianNoise>
 	            <robotNamespace>/</robotNamespace>
 	          </plugin>

File: gazebo_models/velodyne_VLP16/vlp16.urdf.xacro (robot description, xacro)
@@ -1,5 +1,5 @@
 <?xml version="1.0"?>
 <robot xmlns:xacro="http://www.ros.org/wiki/xacro" name="vlp16">
-	<xacro:macro name="vlp16" params="parent name hz *origin">
+	<xacro:macro name="vlp16" params="parent name hz *origin noise:=0.008">
 	    <joint name="${name}_base_mount_joint" type="fixed">
 	      <xacro:insert_block name="origin" />
@@ -35,4 +35,5 @@
     	</link>
 	    <gazebo reference="${name}_link">
+      		<static>true</static>
 	      <turnGravityOff>false</turnGravityOff>
 	      <sensor name='velodyne-VLP16' type='ray'>
@@ -66,9 +67,9 @@
 	          </ray>
 	          <plugin name='gazebo_ros_laser_controller' filename='libgazebo_ros_velodyne_laser.so'>
-	            <topicName>/velodyne_points</topicName>
+	            <topicName>/${name}_points</topicName>
 	            <frameName>${name}</frameName>
 	            <min_range>0.9</min_range>
 	            <max_range>70.0</max_range>
-	            <gaussianNoise>0.008</gaussianNoise>
+	            <gaussianNoise>${noise}</gaussianNoise>
 	            <robotNamespace>/</robotNamespace>
 	          </plugin>
