Commit message: Add hfov and azimuth params to LiDAR xacro models and spawners. Add all launch files for single_sensor calibration tests.

File: gazebo_models/velodyne_HDL32/hdl32.urdf.xacro (robot description, xacro)
@@ -1,5 +1,5 @@
 <?xml version="1.0"?>
 <robot xmlns:xacro="http://www.ros.org/wiki/xacro" name="hdl32">
-	<xacro:macro name="hdl32" params="parent name hz *origin noise:=0.008">
+	<xacro:macro name="hdl32" params="parent name hz *origin noise:=0.008 min_angle:=-180 max_angle:=180 azimuth:=0.2">
 	    <joint name="${name}_base_mount_joint" type="fixed">
 	      <xacro:insert_block name="origin" />
@@ -37,8 +37,8 @@
 	            <scan>
 	              <horizontal>
-	                <samples>1200</samples>
+	                <samples>${(max_angle-min_angle)/azimuth}</samples>
 	                <resolution>1</resolution>
-	                <min_angle>-3.14159</min_angle>
-	                <max_angle>3.14159</max_angle>
+	                <min_angle>${min_angle*3.14159/180}</min_angle>
+	                <max_angle>${max_angle*3.14159/180}</max_angle>
 	              </horizontal>
 	              <vertical>

File: gazebo_models/velodyne_HDL32/hdl32_spawn.urdf.xacro (robot description, xacro)
@@ -5,4 +5,7 @@
   <xacro:arg name="rpy" default="0 0 0" />
   <xacro:arg name="noise" default="0.008" />
+  <xacro:arg name="min_angle" default="-180" />
+  <xacro:arg name="max_angle" default="180" />
+  <xacro:arg name="azimuth" default="0.2" />
   <xacro:arg name="hz" default="1" />
   <xacro:arg name="lidar_name" default="hdl32" />
@@ -30,5 +33,6 @@
     <turnGravityOff>false</turnGravityOff>
   </gazebo>
-  <hdl32 parent="base_footprint" name="$(arg lidar_name)" hz="$(arg hz)" noise="$(arg noise)">
+  <hdl32 parent="base_footprint" name="$(arg lidar_name)" hz="$(arg hz)" noise="$(arg noise)"
+    min_angle="$(arg min_angle)" max_angle="$(arg max_angle)" azimuth="$(arg azimuth)">
     <origin xyz="$(arg xyz)" rpy="$(arg rpy)"/>
   </hdl32>

File: gazebo_models/velodyne_HDL64/hdl64.urdf.xacro (robot description, xacro)
@@ -1,5 +1,5 @@
 <?xml version="1.0"?>
 <robot xmlns:xacro="http://www.ros.org/wiki/xacro" name="hdl64">
-	<xacro:macro name="hdl64" params="parent name hz *origin noise:=0.008">
+	<xacro:macro name="hdl64" params="parent name hz *origin noise:=0.008 min_angle:=-180 max_angle:=180 azimuth:=0.2">
 	    <joint name="${name}_base_mount_joint" type="fixed">
 	      <xacro:insert_block name="origin" />
@@ -31,8 +31,8 @@
 	            <scan>
 	              <horizontal>
-	                <samples>1200</samples>
+	                <samples>${(max_angle-min_angle)/azimuth}</samples>
 	                <resolution>1</resolution>
-	                <min_angle>-3.14159</min_angle>
-	                <max_angle>3.14159</max_angle>
+	                <min_angle>${min_angle*3.14159/180}</min_angle>
+	                <max_angle>${max_angle*3.14159/180}</max_angle>
 	              </horizontal>
 	              <vertical>

File: gazebo_models/velodyne_HDL64/hdl64_spawn.urdf.xacro (robot description, xacro)
@@ -5,4 +5,7 @@
   <xacro:arg name="rpy" default="0 0 0" />
   <xacro:arg name="noise" default="0.008" />
+  <xacro:arg name="min_angle" default="-180" />
+  <xacro:arg name="max_angle" default="180" />
+  <xacro:arg name="azimuth" default="0.2" />
   <xacro:arg name="hz" default="1" />
   <xacro:arg name="lidar_name" default="hdl64" />
@@ -30,5 +33,6 @@
     <turnGravityOff>false</turnGravityOff>
   </gazebo>
-  <hdl64 parent="base_footprint" name="$(arg lidar_name)" hz="$(arg hz)" noise="$(arg noise)">
+  <hdl64 parent="base_footprint" name="$(arg lidar_name)" hz="$(arg hz)" noise="$(arg noise)"
+    min_angle="$(arg min_angle)" max_angle="$(arg max_angle)" azimuth="$(arg azimuth)">
     <origin xyz="$(arg xyz)" rpy="$(arg rpy)"/>
   </hdl64>

File: gazebo_models/velodyne_VLP16/vlp16.urdf.xacro (robot description, xacro)
@@ -1,5 +1,5 @@
 <?xml version="1.0"?>
 <robot xmlns:xacro="http://www.ros.org/wiki/xacro" name="vlp16">
-	<xacro:macro name="vlp16" params="parent name hz *origin noise:=0.008">
+	<xacro:macro name="vlp16" params="parent name hz *origin noise:=0.008 min_angle:=-180 max_angle:=180 azimuth:=0.2">
 	    <joint name="${name}_base_mount_joint" type="fixed">
 	      <xacro:insert_block name="origin" />
@@ -43,8 +43,8 @@
 	            <scan>
 	              <horizontal>
-	                <samples>1200</samples>
+	                <samples>${(max_angle-min_angle)/azimuth}</samples>
 	                <resolution>1</resolution>
-	                <min_angle>-3.14159</min_angle>
-	                <max_angle>3.14159</max_angle>
+	                <min_angle>${min_angle*3.14159/180}</min_angle>
+	                <max_angle>${max_angle*3.14159/180}</max_angle>
 	              </horizontal>
 	              <vertical>

File: gazebo_models/velodyne_VLP16/vlp16_spawn.urdf.xacro (robot description, xacro)
@@ -5,4 +5,7 @@
   <xacro:arg name="rpy" default="0 0 0" />
   <xacro:arg name="noise" default="0.008" />
+  <xacro:arg name="min_angle" default="-180" />
+  <xacro:arg name="max_angle" default="180" />
+  <xacro:arg name="azimuth" default="0.2" />
   <xacro:arg name="hz" default="1" />
   <xacro:arg name="lidar_name" default="vlp16" />
@@ -30,5 +33,6 @@
     <turnGravityOff>false</turnGravityOff>
   </gazebo>
-  <vlp16 parent="base_footprint" name="$(arg lidar_name)" hz="$(arg hz)" noise="$(arg noise)">
+  <vlp16 parent="base_footprint" name="$(arg lidar_name)" hz="$(arg hz)" noise="$(arg noise)"
+    min_angle="$(arg min_angle)" max_angle="$(arg max_angle)" azimuth="$(arg azimuth)">
     <origin xyz="$(arg xyz)" rpy="$(arg rpy)"/>
   </vlp16>
